File: eletronica/seguidor.kicad_pcb (KiCad board)
At the start: 2 copper layers, 28 parts, among them M1 INDUCTOR, M2 INDUCTOR, U1 LM324

Commit message: Almost
Parts:
- added Power: Battery, Pin_Headers:Pin_Header_Straight_2x01, F.Cu at (166.4, 83.8)
- moved R5 102.4 mm to (157.5, 57.1), turned to 180 degrees
- moved R3 100.6 mm to (157.5, 49.5), turned to 180 degrees
- moved C1 87.1 mm to (165.1, 57.1)
- moved R2 74.8 mm to (157.5, 66.0)
- moved R1 70.8 mm to (167.6, 72.4)
- moved D2 67.1 mm to (174.0, 121.9), turned to 90 degrees
- moved R6 64.2 mm to (144.8, 111.8), turned to 270 degrees
- moved C3 58.6 mm to (132.1, 81.3)
- moved R4 58.4 mm to (129.5, 69.8), turned to 90 degrees
- moved C2 53.6 mm to (143.5, 71.1), turned to 0 degrees
- moved U1 44.0 mm to (160.0, 81.3), turned to 270 degrees
- moved LED1 42.2 mm to (146.1, 128.3)
- moved D1 39.8 mm to (130.8, 121.9), turned to 90 degrees
- moved M2 38.6 mm to (180.3, 118.1), turned to 90 degrees
- moved LED2 36.3 mm to (158.8, 128.3)
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Routing:
- net GND: track 0.00 -> 243.6 mm
- net VCC: track 0.00 -> 216.9 mm
- net Net-(C1-Pad1): track 0.00 -> 138.4 mm
- net Net-(LDR2-Pad1): track 0.00 -> 78.9 mm
- net Net-(R3-Pad2): track 0.00 -> 61.4 mm
- net Net-(R3-Pad1): track 0.00 -> 49.7 mm
- net Net-(C2-Pad1): track 0.00 -> 25.2 mm
- net Net-(C2-Pad2): track 0.00 -> 25.1 mm
- net Net-(C5-Pad2): track 0.00 -> 22.3 mm
- net Net-(C6-Pad2): track 0.00 -> 22.3 mm
- net Net-(LDR1-Pad1): track 0.00 -> 13.5 mm
- net Net-(R8-Pad2): track 0.00 -> 8.45 mm
- net Net-(R9-Pad1): track 0.00 -> 8.45 mm
- net Net-(LED1-Pad2): track 0.00 -> 6.88 mm
- net Net-(LED2-Pad2): track 0.00 -> 6.88 mm
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Other:
- net class Default: clearance 0.2 -> 0.5; trace_width 0.6096 -> 0.7
- net class POWER added: clearance 0.2, trace_width 0.8, via_dia 0.6, via_drill 0.4
- rule trace_clearance: 0.2 -> 0.5

Commit message: ALMOSSSST!
Routing:
- net GND: track 243.6 -> 257.6 mm
- net Net-(C2-Pad1): track 25.2 -> 38.9 mm
Changed lines of the file:
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@@
   (general
     (links 55)
-    (no_connects 5)
-    (area 115.065199 44.595 185.924802 143.235)
+    (no_connects 3)
+    (area 117.935 44.295 185.000002 143.535)
     (thickness 1.6)
     (drawings 0)
-    (tracks 143)
+    (tracks 151)
     (zones 0)
     (modules 29)
@@
   (segment (start 157.48 66.04) (end 157.48 72.39) (width 0.6096) (layer B.Cu) (net 1))
   (segment (start 157.48 72.39) (end 157.48 81.28) (width 0.6096) (layer B.Cu) (net 1))
-  (segment (start 139.7 106.68) (end 139.7 104.14) (width 0.7) (layer B.Cu) (net 2))
+  (segment (start 139.7 91.44) (end 139.7 105.41) (width 0.7) (layer B.Cu) (net 2))
+  (segment (start 139.7 106.68) (end 139.7 105.41) (width 0.7) (layer B.Cu) (net 2))
+  (segment (start 142.24 101.6) (end 162.56 101.6) (width 0.7) (layer B.Cu) (net 2))
+  (segment (start 139.7 104.14) (end 142.24 101.6) (width 0.7) (layer B.Cu) (net 2))
+  (segment (start 139.7 105.41) (end 139.7 104.14) (width 0.7) (layer B.Cu) (net 2))
   (segment (start 165.1 104.14) (end 165.1 106.68) (width 0.7) (layer B.Cu) (net 2))
   (segment (start 162.56 101.6) (end 165.1 104.14) (width 0.7) (layer B.Cu) (net 2))
-  (segment (start 142.24 101.6) (end 162.56 101.6) (width 0.7) (layer B.Cu) (net 2))
-  (segment (start 139.7 104.14) (end 142.24 101.6) (width 0.7) (layer B.Cu) (net 2))
   (segment (start 158.75 137.16) (end 158.75 138.43) (width 0.7) (layer B.Cu) (net 2))
   (segment (start 184.15 100.33) (end 170.18 86.36) (width 0.7) (layer B.Cu) (net 2))
@@
   (segment (start 142.24 86.36) (end 149.86 86.36) (width 0.7) (layer B.Cu) (net 2))
   (segment (start 149.86 86.36) (end 152.4 88.9) (width 0.7) (layer B.Cu) (net 2))
+  (segment (start 154.94 88.9) (end 154.94 92.71) (width 0.7) (layer B.Cu) (net 3))
+  (segment (start 149.86 92.71) (end 149.86 88.9) (width 0.7) (layer B.Cu) (net 3))
+  (segment (start 151.13 93.98) (end 149.86 92.71) (width 0.7) (layer B.Cu) (net 3))
+  (segment (start 153.67 93.98) (end 151.13 93.98) (width 0.7) (layer B.Cu) (net 3))
+  (segment (start 154.94 92.71) (end 153.67 93.98) (width 0.7) (layer B.Cu) (net 3))
   (segment (start 129.54 69.85) (end 142.24 69.85) (width 0.6096) (layer B.Cu) (net 3))
   (segment (start 142.24 69.85) (end 143.51 71.12) (width 0.6096) (layer B.Cu) (net 3))
-  (segment (start 143.51 71.12) (end 143.51 80.01) (width 0.6096) (layer B.Cu) (net 3))
+  (segment (start 143.51 71.12) (end 143.51 76.2) (width 0.6096) (layer B.Cu) (net 3))
+  (segment (start 143.51 76.2) (end 143.51 80.01) (width 0.6096) (layer B.Cu) (net 3))
   (segment (start 143.51 80.01) (end 144.78 81.28) (width 0.6096) (layer B.Cu) (net 3))
   (segment (start 147.32 57.15) (end 147.32 69.93) (width 0.6096) (layer B.Cu) (net 4))
@@
   (segment (start 148.51 71.12) (end 148.51 80.09) (width 0.6096) (layer B.Cu) (net 4))
   (segment (start 148.51 80.09) (end 147.32 81.28) (width 0.6096) (layer B.Cu) (net 4))
+  (segment (start 144.78 111.76) (end 144.78 110.49) (width 0.7) (layer B.Cu) (net 5))
+  (segment (start 144.78 110.49) (end 146.05 109.22) (width 0.7) (layer B.Cu) (net 5))
+  (segment (start 146.05 109.22) (end 157.48 109.22) (width 0.7) (layer B.Cu) (net 5))
+  (segment (start 157.48 109.22) (end 160.02 111.76) (width 0.7) (layer B.Cu) (net 5))
   (segment (start 135.89 83.82) (end 135.89 80.01) (width 0.7) (layer B.Cu) (net 5))
   (segment (start 121.92 115.57) (end 124.46 118.11) (width 0.7) (layer B.Cu) (net 5))
@@
   (segment (start 167.64 119.38) (end 167.64 132.08) (width 0.7) (layer B.Cu) (net 5))
   (segment (start 160.02 111.76) (end 167.64 119.38) (width 0.7) (layer B.Cu) (net 5))
-  (segment (start 144.78 111.76) (end 144.78 110.49) (width 0.7) (layer B.Cu) (net 5))
-  (segment (start 157.48 109.22) (end 160.02 111.76) (width 0.7) (layer B.Cu) (net 5))
-  (segment (start 146.05 109.22) (end 157.48 109.22) (width 0.7) (layer B.Cu) (net 5))
-  (segment (start 144.78 110.49) (end 146.05 109.22) (width 0.7) (layer B.Cu) (net 5))
   (segment (start 137.16 119.38) (end 144.78 111.76) (width 0.7) (layer B.Cu) (net 5))
   (segment (start 130.80746 121.91948) (end 134.62052 121.91948) (width 0.7) (layer B.Cu) (net 5))

Commit message: done
Parts:
- removed Power: Battery, Pin_Headers:Pin_Header_Straight_2x01
- added PWR: Battery, Pin_Headers:Pin_Header_Straight_2x01, F.Cu at (165.7, 83.8)
- added REF**: Pin_Header_Straight_1x01, Pin_Headers:Pin_Header_Straight_1x01, F.Cu at (149.2, 99.1)
- added REF**: Pin_Header_Straight_1x01, Pin_Headers:Pin_Header_Straight_1x01, F.Cu at (152.4, 99.1)
- added REF**: Pin_Header_Straight_1x01, Pin_Headers:Pin_Header_Straight_1x01, F.Cu at (149.2, 128.3)
- added REF**: Pin_Header_Straight_1x01, Pin_Headers:Pin_Header_Straight_1x01, F.Cu at (152.4, 128.3)
Routing:
- net Net-(C2-Pad1): track 38.9 -> 186.2 mm
- net Net-(LDR1-Pad1): track 13.5 -> 78.5 mm
- net Net-(C1-Pad1): track 138.4 -> 145.4 mm
- added copper zone on B.Cu, net GND
Other:
- board outline added: 72.4 x 99.7 mm
